File: PCB/20190213.brd (EAGLE design)
At the start: 100 x 80 mm, 3 parts, among them Q1 60V/32A/35mΩ, Q2 60V/32A/35mΩ

Commit message: DB init and PCB init.
Parts:
- added AIR1, AIR2, AIR3, IN_12V, IN_24V, IN_9V, OUT_12V, OUT_12V1, OUT_12V2, OUT_24V, OUT_9V, OUT_9V1, OUT_9V2: (no value), SparkFun-Connectors:MOLEX-1X2_LOCK
- added C1: 10uF, SparkFun-Capacitors:CPOL-RADIAL-2.5MM-5MM-KIT
- added D1, D2, D3: (no value), SparkFun-LED:LED_5MM
- added JP1, JP2: JUMPER-SMT_2_NC_PASTE_SILK, SparkFun-Jumpers:SMT-JUMPER_2_NC_PASTE_SILK
- added JP3, JP4: JUMPER-SMT_3_NO_NO-SILK, SparkFun-Jumpers:SMT-JUMPER_3_NO_NO-SILK
- added LOGO1: ROHS_LOGO, SparkFun-Aesthetics:ROHS_LOGO_0.18_IN
- added OK1, OK2, OK3: PC817, optocoupler:DIL04
- added R1, R2, R3, R4, R5, R6, R7, R8: 10M, SparkFun-Resistors:AXIAL-0.3
- added T1, T2, T3: 2N6292, transistor:TO220
- moved Q2 109.5 mm to (73.7, 76.2)
- moved Q1 85.2 mm to (-19.1, 77.5)
- moved MEGA2560PRO1 8.98 mm to (36.8, 50.8)
Connections:
- new net +12V: IN_12V.1, OUT_12V.1, OUT_12V1.1, OUT_12V2.1
- new net +24V: AIR1.1, AIR2.1, AIR3.1, IN_24V.1, OUT_24V.1
- new net +5V: MEGA2560PRO1.5V@3, OK1.4, OK2.4, OK3.4
- new net +9V: IN_9V.1, OUT_9V.1, OUT_9V1.1, OUT_9V2.1
- new net 3.3V: MEGA2560PRO1.3V3@2, R8.P$2
- new net GND: IN_12V.2, IN_24V.2, IN_9V.2, OK1.2, OK2.2, OK3.2, OUT_12V.2, OUT_12V1.2, OUT_12V2.2, OUT_24V.2, OUT_9V.2, OUT_9V1.2, OUT_9V2.2, R7.P$2, T1.3, T2.3, T3.3
- new net N$1: R1.P$2, T1.1
- new net N$10: R6.P$2, T1.2
- new net N$11: R5.P$2, T2.2
- new net N$12: R4.P$2, T3.2
- new net N$13: C1.1, MEGA2560PRO1.RESET, R8.P$1
- new net N$14: C1.2, R7.P$1
- new net N$15: MEGA2560PRO1.D10, OK1.1
- new net N$16: MEGA2560PRO1.D12, OK2.1
- new net N$17: MEGA2560PRO1.D14, OK3.1
- new net N$2: R2.P$2, T2.1
- new net N$3: R3.P$2, T3.1
- new net N$4: AIR1.2, R4.P$1
- new net N$5: AIR2.2, R5.P$1
- new net N$6: AIR3.2, R6.P$1
- new net N$7: OK1.3, R1.P$1
- new net N$8: OK2.3, R2.P$1
- new net N$9: OK3.3, R3.P$1
Other:
- board size 100 x 80 mm -> 160 x 100 mm
