File: PCB/20190213.sch (EAGLE design)
At the start: 3 parts, among them Q1 60V/32A/35mΩ, Q2 60V/32A/35mΩ

Commit message: DB init and PCB init.
Parts:
- added AIR1, AIR2, AIR3, IN_12V, IN_24V, IN_9V, OUT_12V, OUT_12V1, OUT_12V2, OUT_24V, OUT_9V, OUT_9V1, OUT_9V2: (no value), SparkFun-Connectors:CONN_02POLAR_LOCK
- added C1: 10uF, SparkFun-Capacitors:10UF-POLAR-RADIAL-2.5MM-KIT-25V-20%
- added D1, D2, D3: (no value), SparkFun-LED:LED5MM
- added JP1, JP2: JUMPER-SMT_2_NC_PASTE_SILK, SparkFun-Jumpers:JUMPER-SMT_2_NC_PASTE_SILK
- added JP3, JP4: JUMPER-SMT_3_NO_NO-SILK, SparkFun-Jumpers:JUMPER-SMT_3_NO_NO-SILK
- added LOGO1: ROHS_LOGO, SparkFun-Aesthetics:ROHS_LOGO
- added OK1, OK2, OK3: PC817, optocoupler:PC817
- added R1, R2, R3, R4, R5, R6, R7, R8: 10M, SparkFun-Resistors:10MOHM-HORIZ-1/4W-5%
- added T1, T2, T3: 2N6292, transistor:2N6292
Connections:
- new net +12V: IN_12V.1, OUT_12V.1, OUT_12V1.1, OUT_12V2.1
- new net +24V: AIR1.1, AIR2.1, AIR3.1, IN_24V.1, OUT_24V.1
- new net +5V: MEGA2560PRO1.5V@3, OK1.COL, OK2.COL, OK3.COL
- new net +9V: IN_9V.1, OUT_9V.1, OUT_9V1.1, OUT_9V2.1
- new net 3.3V: MEGA2560PRO1.3V3@2, R8.2
- new net GND: IN_12V.2, IN_24V.2, IN_9V.2, OK1.C, OK2.C, OK3.C, OUT_12V.2, OUT_12V1.2, OUT_12V2.2, OUT_24V.2, OUT_9V.2, OUT_9V1.2, OUT_9V2.2, R7.2, T1.E, T2.E, T3.E
- new net N$1: R1.2, T1.B
- new net N$10: R6.2, T1.C
- new net N$11: R5.2, T2.C
- new net N$12: R4.2, T3.C
- new net N$13: C1.+, MEGA2560PRO1.RESET, R8.1
- new net N$14: C1.-, R7.1
- new net N$15: MEGA2560PRO1.D10, OK1.A
- new net N$16: MEGA2560PRO1.D12, OK2.A
- new net N$17: MEGA2560PRO1.D14, OK3.A
- new net N$2: R2.2, T2.B
- new net N$3: R3.2, T3.B
- new net N$4: AIR1.2, R4.1
- new net N$5: AIR2.2, R5.1
- new net N$6: AIR3.2, R6.1
- new net N$7: OK1.EMIT, R1.1
- new net N$8: OK2.EMIT, R2.1
- new net N$9: OK3.EMIT, R3.1
Other:
- moved on the sheet: Q1, Q2
