File: PCB/20190501.brd (EAGLE design)
At the start: 160 x 63.5 mm, 49 parts, among them J1 POWER_JACK, J2 POWER_JACK, Q1 BD437, Q2 BD437, Q3 BD437

Commit message: fix PCB wire
Parts:
- removed HYVISION: W5500, DECADE2019:W5500
- added LOGO1: ROHS_LOGO, SparkFun-Aesthetics:ROHS_LOGO_0.18_IN
- added U$1: W5500, DECADE2019:W5500
- moved JP6 9.50 mm to (33.0, 2.50)
- moved JP5 4.30 mm to (36.0, 6.00)
Connections:
- removed net N$38: HYVISION.MOSI, JP5.2
- new net N$32: MEGA2560PRO1.SCK, U$1.SCLK
- net +5V: now also U$1.5V; no longer HYVISION.5V
- net GND: now also U$1.GND; no longer HYVISION.GND
- net N$13: now also U$1.RST; no longer HYVISION.RST
- net N$31: now also JP5.2, U$1.MOSI; no longer HYVISION.SCLK, MEGA2560PRO1.SCK
- net N$33: now also U$1.SCS; no longer HYVISION.SCS
- net N$37: now also U$1.MISO; no longer HYVISION.MISO
Routing:
- net N$32: track 0.00 -> 53.0 mm, vias 1 -> 0
- net GND: track 546.3 -> 579.7 mm
- net N$13: track 124.0 -> 153.0 mm
- net +5V: track 392.0 -> 366.2 mm
- net N$38: track 18.0 -> 0.00 mm
- net N$31: track 46.4 -> 31.9 mm
- net N$33: track 37.9 -> 51.4 mm
- net N$37: track 23.1 -> 15.5 mm, vias 1 -> 0
- net N$30: track 32.4 -> 28.5 mm
- net N$36: track 27.1 -> 28.2 mm
- net N$28: track 138.9 -> 139.6 mm
