File: PCB/2020/sdcard_noBMP.brd (EAGLE design)
At the start: 108 x 86.5 mm, 23 parts, among them J1 CONN_20X2NOSILK, J2 CONN_20X2NOSILK, J3 CONN_20X2NOSILK, J4 CONN_20X2NOSILK, X1 JST-XH-12-PIN-LONG-PAD, X2 JST-XH-06-PIN-LONG-PAD, X3 JST-XH-06-PIN-LONG-PAD, X4 JST-XH-12-PIN-LONG-PAD

Commit message: PCB update
Connections:
- removed net N$9: JP1.1, JP2.1, JP3.3, R_5V_BUFF.2
- new net N$1: JP1.1, JP2.1, JP3.3, R_5V_BUFF.2, U$1./RST, U$1./SLP
- net N$14: no longer U$1./RST, U$1./SLP
Routing:
- net N$1: track 0.00 -> 22.8 mm
- net N$9: track 13.3 -> 0.00 mm
- net N$14: track 23.2 -> 15.3 mm
Other:
- board text added: "Xception_V0.9.0"
- board text removed: "HY_Vision_V0318"
